File: Kicad/HVPSController2/HVPSController2.kicad_sch (KiCad schematic)
At the start: 191 parts, among them J1 Vsupply, J10 Conn_01x02_Pin, J11 USB RWGBS, J12 USB RWGBS, J13 Conn_01x01_Pin, J14 Conn_01x01_Pin, J15 Tap, J16 Conn_01x02_Pin, J17 Conn_01x02_Pin, J2 GND, J20 Standoff Hole, J21 Standoff Hole, J22 Standoff Hole, J23 Standoff Hole, J24 Conn_01x02_Pin, J25 Standoff Hole, J26 Standoff Hole, J3 Snubber, J32 Conn_01x02_Pin, J33 Conn_01x02_Pin, J34 Conn_01x02_Pin, J35 Conn_01x02_Pin, J36 Conn_01x02_Pin, J4 Conn_01x08_Pin, J5 Snubber, J6 Snubber, J7 Snubber, J8 SCL, SDA, +, GND, J9 Tap

Commit message: Going great, debugging villard now works!
Parts:
- C81: value 0.1uF -> 10nF
- C82: value 0.1uF -> 22nF
Changed lines of the file:
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@@
 			)
 		)
-		(property "Value" "0.1uF"
+		(property "Value" "22nF"
 			(at 230.378 260.35 90)
 			(effects
@@
 			)
 		)
-		(property "Value" "0.1uF"
+		(property "Value" "10nF"
 			(at 123.698 334.01 90)
 			(effects
